File: Function.kicad_sch (KiCad schematic)
At the start: 0 parts

Commit message: Power Supply
Parts:
- added C16, C18: 0.1u, Capacitor_THT:C_Disc_D4.7mm_W2.5mm_P5.00mm, symbol Device:C
- added C17, C19: 1u, Capacitor_THT:C_Disc_D4.7mm_W2.5mm_P5.00mm, symbol Device:C
- added J63: Screw_Terminal_01x03, TerminalBlock_Phoenix:TerminalBlock_Phoenix_PT-1,5-3-5.0-H_1x03_P5.00mm_Horizontal, symbol Connector:Screw_Terminal_01x03
- added R45, R46: 120, Resistor_THT:R_Axial_DIN0207_L6.3mm_D2.5mm_P10.16mm_Horizontal, symbol Device:R_US
- added RV6: 47k, Potentiometer_THT:Potentiometer_Alps_RK163_Dual_Horizontal, symbol Device:R_Potentiometer_Dual
- added U5: LM324, Package_DIP:DIP-14_W7.62mm_LongPads, symbol Amplifier_Operational:LM324
- added U6: LM317_TO-220, Package_TO_SOT_THT:TO-220-3_Vertical, symbol Regulator_Linear:LM317_TO-220
- added U7: LM337_TO252, Package_TO_SOT_SMD:TO-252-2, symbol Regulator_Linear:LM337_TO252
Connections:
- new net: C18.1, J63.3 (Pin_3), U6.3 (VI)
- new net: R46.2, RV6.6, U6.1 (ADJ)
- new net: R45.1, RV6.1, U7.1 (ADJ)
- new net: C16.2, J63.1 (Pin_1), U7.2 (VI)
- new net +15V: C19.1, R46.1, U6.2 (VO)
- new net -15V: C17.2, R45.2, U7.3 (VO)
- new net GND: C16.1, C17.1, C18.2, C19.2, J63.2 (Pin_2), RV6.2, RV6.3, RV6.4, RV6.5
Other:
- note added: "POWER SUPPLY"

Commit message: Floor Planning 50%
Parts:
- removed U5: LM324, Package_DIP:DIP-14_W7.62mm_LongPads, symbol Amplifier_Operational:LM324
- added J39, J66, J67: Conn_02x04_Counter_Clockwise, Connector_PinHeader_2.54mm:PinHeader_2x04_P2.54mm_Vertical, symbol Connector_Generic:Conn_02x04_Counter_Clockwise
- C16, C18, R45, R46, RV6, U6, U7: now not fitted; now left out of the parts list
- C17, C19: value 1u -> 0.1u; now not fitted; now left out of the parts list
Connections:
- net +15V: now also C18.1, J63.3 (Pin_3), U6.3 (VI), J67.1 (Pin_1), J67.2 (Pin_2), J67.3 (Pin_3), J67.4 (Pin_4), J67.5 (Pin_5), J67.6 (Pin_6), J67.7 (Pin_7), J67.8 (Pin_8)
- net -15V: now also C16.2, J63.1 (Pin_1), U7.2 (VI), J66.1 (Pin_1), J66.2 (Pin_2), J66.3 (Pin_3), J66.4 (Pin_4), J66.5 (Pin_5), J66.6 (Pin_6), J66.7 (Pin_7), J66.8 (Pin_8)
- net GND: now also RV6.1, J39.1 (Pin_1), J39.2 (Pin_2), J39.3 (Pin_3), J39.4 (Pin_4), J39.5 (Pin_5), J39.6 (Pin_6), J39.7 (Pin_7), J39.8 (Pin_8); no longer RV6.3
- net at R45.1, U7.1 (ADJ): now also RV6.3; no longer RV6.1
Other:
- note added: "Ground Plane"
- moved on the sheet: J63
