File: Inverting.kicad_sch (KiCad schematic)
At the start: 0 parts

Commit message: added inverting ckt
Parts:
- added C4, C8, C9: C, Capacitor_THT:C_Disc_D5.0mm_W2.5mm_P5.00mm, symbol Device:C
- added J40, J41, J42, J43, J44, J45, J46, J47, J48, J49, J50: Conn_01x04_Pin, Connector_PinHeader_2.54mm:PinHeader_1x04_P2.54mm_Vertical, symbol Connector:Conn_01x04_Pin
- added R21, R22, R23, R24, R25: R_US, Resistor_THT:R_Axial_DIN0207_L6.3mm_D2.5mm_P10.16mm_Horizontal, symbol Device:R_US
- added RV1: R_Potentiometer_Trim_US, Potentiometer_THT:Potentiometer_Runtron_RM-065_Vertical, symbol Device:R_Potentiometer_Trim_US
- added U2: LM741, Package_DIP:DIP-8_W7.62mm_LongPads, symbol Amplifier_Operational:LM741
Connections:
- new net: J50.1 (Pin_1), J50.2 (Pin_2), J50.3 (Pin_3), J50.4 (Pin_4), R21.1
- new net: C8.2, J44.1 (Pin_1), J44.2 (Pin_2), J44.3 (Pin_3), J44.4 (Pin_4)
- new net: C4.1, C8.1, C9.1, J40.1 (Pin_1), J40.2 (Pin_2), J40.3 (Pin_3), J40.4 (Pin_4), R21.2, R22.2, R23.2, R24.2, R25.1, U2.3 (+)
- new net: C9.2, J45.1 (Pin_1), J45.2 (Pin_2), J45.3 (Pin_3), J45.4 (Pin_4)
- new net: RV1.2, U2.1 (NULL)
- new net: RV1.3, U2.5 (NULL)
- new net: J47.1 (Pin_1), J47.2 (Pin_2), J47.3 (Pin_3), J47.4 (Pin_4), R24.1
- new net: J46.1 (Pin_1), J46.2 (Pin_2), J46.3 (Pin_3), J46.4 (Pin_4), R25.2
- new net: J49.1 (Pin_1), J49.2 (Pin_2), J49.3 (Pin_3), J49.4 (Pin_4), R22.1
- new net: J48.1 (Pin_1), J48.2 (Pin_2), J48.3 (Pin_3), J48.4 (Pin_4), R23.1
- new net: J42.1 (Pin_1), J42.2 (Pin_2), J42.3 (Pin_3), J42.4 (Pin_4), U2.6
- new net: C4.2, J43.1 (Pin_1), J43.2 (Pin_2), J43.3 (Pin_3), J43.4 (Pin_4)
- new net +15V: U2.7 (V+)
- new net -15V: U2.4 (V-)
- new net GND: J41.1 (Pin_1), J41.2 (Pin_2), J41.3 (Pin_3), J41.4 (Pin_4), U2.2 (-)
- no-connect marks 0 -> 1
Other:
- note added: "Inverted Op-Amp"

Commit message: Added fetures
Parts:
- RV1: value R_Potentiometer_Trim_US -> 10k
Connections:
- net GND: now also U2.3 (+); no longer U2.2 (-)
- net at C4.1, C8.1, C9.1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: now also U2.2 (-); no longer U2.3 (+)
- net at RV1.2: now also U2.5 (NULL); no longer U2.1 (NULL)
- net at RV1.3: now also U2.1 (NULL); no longer U2.5 (NULL)
Other:
- moved on the sheet: RV1
Changed lines of the file:
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@@
 	)
 	(no_connect
-		(at 157.48 123.19)
+		(at 157.48 102.87)
 	)
 	(wire
@@
 	(wire
 		(pts
+			(xy 153.67 99.06) (xy 153.67 100.33)
+		)
+		(stroke
+			(width 0)
+			(type default)
+		)
+	)
+	(wire
+		(pts
 			(xy 111.76 76.2) (xy 114.3 76.2)
 		)
@@
 	(wire
 		(pts
-			(xy 153.67 119.38) (xy 151.13 119.38)
-		)
-		(stroke
-			(width 0)
-			(type default)
-		)
-	)
-	(wire
-		(pts
 			(xy 109.22 63.5) (xy 111.76 63.5)
 		)
@@
 	(wire
 		(pts
-			(xy 148.59 99.06) (xy 148.59 100.33)
+			(xy 151.13 95.25) (xy 151.13 100.33)
 		)
 		(stroke
@@
 	(wire
 		(pts
-			(xy 153.67 115.57) (xy 157.48 115.57)
+			(xy 151.13 95.25) (xy 157.48 95.25)
 		)
 		(stroke
@@
 	(wire
 		(pts
+			(xy 148.59 115.57) (xy 148.59 118.11)
+		)
+		(stroke
+			(width 0)
+			(type default)
+		)
+	)
+	(wire
+		(pts
 			(xy 170.18 107.95) (xy 172.72 107.95)
 		)
@@
 	(wire
 		(pts
-			(xy 151.13 115.57) (xy 151.13 119.38)
-		)
-		(stroke
-			(width 0)
-			(type default)
-		)
-	)
-	(wire
-		(pts
 			(xy 170.18 50.8) (xy 172.72 50.8)
 		)
@@
 	(wire
 		(pts
-			(xy 148.59 115.57) (xy 148.59 116.84)
-		)
-		(stroke
-			(width 0)
-			(type default)
-		)
-	)
-	(wire
-		(pts
 			(xy 152.4 63.5) (xy 165.1 63.5)
 		)
@@
 		(pts
 			(xy 167.64 88.9) (xy 170.18 88.9)
+		)
+		(stroke
+			(width 0)
+			(type default)
+		)
+	)
+	(wire
+		(pts
+			(xy 148.59 97.79) (xy 148.59 100.33)
 		)
 		(stroke
@@
 	(symbol
 		(lib_id "Device:R_Potentiometer_Trim_US")
-		(at 157.48 119.38 180)
-		(unit 1)
-		(exclude_from_sim no)
-		(in_bom yes)
-		(on_board yes)
-		(dnp no)
-		(fields_autoplaced yes)
+		(at 157.48 99.06 180)
+		(unit 1)
+		(exclude_from_sim no)
+		(in_bom yes)
+		(on_board yes)
+		(dnp no)
 		(property "Reference" "RV1"
-			(at 160.02 118.1099 0)
+			(at 158.75 101.854 0)
 			(effects
 				(font
@@
 			)
 		)
-		(property "Value" "R_Potentiometer_Trim_US"
-			(at 160.02 120.6499 0)
+		(property "Value" "10k"
+			(at 157.988 94.234 0)
 			(effects
 				(font
@@
 		)
 		(property "Footprint" "Potentiometer_THT:Potentiometer_Runtron_RM-065_Vertical"
-			(at 157.48 119.38 0)
+			(at 157.48 99.06 0)
 			(effects
 				(font
@@
 		)
 		(property "Datasheet" "~"
-			(at 157.48 119.38 0)
+			(at 157.48 99.06 0)
 			(effects
 				(font
@@
 		)
 		(property "Description" "Trim-potentiometer, US symbol"
-			(at 157.48 119.38 0)
+			(at 157.48 99.06 0)
 			(effects
 				(font
@@
 	(symbol
 		(lib_id "power:+15V")
-		(at 148.59 99.06 0)
-		(unit 1)
-		(exclude_from_sim no)
-		(in_bom yes)
-		(on_board yes)
-		(dnp no)
-		(fields_autoplaced yes)
+		(at 148.59 118.11 180)
+		(unit 1)
+		(exclude_from_sim no)
+		(in_bom yes)
+		(on_board yes)
+		(dnp no)
 		(property "Reference" "#PWR03"
-			(at 148.59 102.87 0)
+			(at 148.59 114.3 0)
 			(effects
 				(font
@@
 		)
 		(property "Value" "+15V"
-			(at 148.59 93.98 0)
-			(effects
-				(font
-					(size 1.27 1.27)
-				)
+			(at 145.288 122.428 0)
+			(effects
+				(font
+					(size 1.27 1.27)
+				)
+				(justify right)
 			)
 		)
 		(property "Footprint" ""
-			(at 148.59 99.06 0)
+			(at 148.59 118.11 0)
 			(effects
 				(font
@@
 		)
 		(property "Datasheet" ""
-			(at 148.59 99.06 0)
+			(at 148.59 118.11 0)
 			(effects
 				(font
@@
 		)
 		(property "Description" "Power symbol creates a global label with name \"+15V\""
-			(at 148.59 99.06 0)
+			(at 148.59 118.11 0)
 			(effects
 				(font
@@
 	(symbol
 		(lib_id "power:-15V")
-		(at 148.59 116.84 180)
-		(unit 1)
-		(exclude_from_sim no)
-		(in_bom yes)
-		(on_board yes)
-		(dnp no)
-		(fields_autoplaced yes)
+		(at 148.59 97.79 0)
+		(unit 1)
+		(exclude_from_sim no)
+		(in_bom yes)
+		(on_board yes)
+		(dnp no)
 		(property "Reference" "#PWR04"
-			(at 148.59 113.03 0)
+			(at 148.59 101.6 0)
 			(effects
 				(font
@@
 		)
 		(property "Value" "-15V"
-			(at 148.59 121.92 0)
-			(effects
-				(font
-					(size 1.27 1.27)
-				)
+			(at 142.748 95.758 0)
+			(effects
+				(font
+					(size 1.27 1.27)
+				)
+				(justify left)
 			)
 		)
 		(property "Footprint" ""
-			(at 148.59 116.84 0)
+			(at 148.59 97.79 0)
 			(effects
 				(font
@@
 		)
 		(property "Datasheet" ""
-			(at 148.59 116.84 0)
+			(at 148.59 97.79 0)
 			(effects
 				(font
@@
 		)
 		(property "Description" "Power symbol creates a global label with name \"-15V\""
-			(at 148.59 116.84 0)
+			(at 148.59 97.79 0)
 			(effects
 				(font
@@
 		(lib_id "Amplifier_Operational:LM741")
 		(at 151.13 107.95 0)
+		(mirror x)
 		(unit 1)
 		(exclude_from_sim no)
@@
 		(dnp no)
 		(property "Reference" "U2"
-			(at 153.924 100.584 0)
+			(at 153.924 115.316 0)
 			(effects
 				(font
@@
 		)
 		(property "Value" "LM741"
-			(at 154.432 103.378 0)
+			(at 154.432 112.522 0)
 			(effects
 				(font
@@
 		)
 		(property "Footprint" "Package_DIP:DIP-8_W7.62mm_LongPads"
-			(at 152.4 106.68 0)
+			(at 152.4 109.22 0)
 			(effects
 				(font
@@
 		)
 		(property "Datasheet" "http://www.ti.com/lit/ds/symlink/lm741.pdf"
-			(at 154.94 104.14 0)
+			(at 154.94 111.76 0)
 			(effects
 				(font
@@
 		(on_board yes)
 		(dnp no)
-		(fields_autoplaced yes)
 		(property "Reference" "J42"
-			(at 168.91 97.79 90)
+			(at 175.768 105.664 90)
 			(effects
 				(font
@@
 		)
 		(property "Value" "Conn_01x04_Pin"
-			(at 168.91 100.33 90)
-			(effects
-				(font
+			(at 169.418 109.474 90)
+			(effects
+				(font

Commit message: Power Supply
Parts:
- C4: value C -> 1u
- C8: value C -> 0.1u
- C9: value C -> 0.01u
- R21: value R_US -> 1k
- R22: value R_US -> 2.2k
- R23: value R_US -> 4.7k
- R24: value R_US -> 5.6k
- R25: value R_US -> 10k
Changed lines of the file:
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@@
 			)
 		)
-		(property "Value" "C"
+		(property "Value" "0.01u"
 			(at 148.59 58.42 90)
 			(effects
@@
 	)
 	(symbol
+		(lib_name "R_US_1")
 		(lib_id "Device:R_US")
 		(at 130.81 88.9 90)
@@
 			)
 		)
-		(property "Value" "R_US"
+		(property "Value" "1k"
 			(at 130.81 85.09 90)
 			(effects
@@
 			)
 		)
-		(property "Value" "R_US"
+		(property "Value" "10k"
 			(at 148.59 46.99 90)
 			(effects
@@
 			)
 		)
-		(property "Value" "R_US"
+		(property "Value" "2.2k"
 			(at 130.81 72.39 90)
 			(effects
@@
 			)
 		)
-		(property "Value" "R_US"
+		(property "Value" "4.7k"
 			(at 130.81 59.69 90)
 			(effects
@@
 			)
 		)
-		(property "Value" "C"
+		(property "Value" "0.1u"
 			(at 148.59 71.12 90)
 			(effects
@@
 			)
 		)
-		(property "Value" "R_US"
+		(property "Value" "5.6k"
 			(at 130.81 46.99 90)
 			(effects
@@
 			)
 		)
-		(property "Value" "C"
+		(property "Value" "1u"
 			(at 148.59 83.82 90)
 			(effects

Commit message: Floor Planning 50%
Parts:
- C4, C8, C9: footprint Capacitor_THT:C_Disc_D5.0mm_W2.5mm_P5.00mm -> Capacitor_SMD:C_0805_2012Metric_Pad1.18x1.45mm_HandSolder
- RV1: footprint Potentiometer_THT:Potentiometer_Runtron_RM-065_Vertical -> Potentiometer_THT:Potentiometer_Bourns_3296W_Vertical
Connections:
- net -15V: now also RV1.2
- net at RV1.1: now also U2.1 (NULL)
- net at U2.5 (NULL): now also RV1.3; no longer RV1.2
- no-connect marks 1 -> 0
Other:
- moved on the sheet: RV1
Changed lines of the file:
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@@
 		(color 0 0 0 0)
 	)
-	(no_connect
-		(at 157.48 102.87)
-	)
 	(wire
 		(pts
@@
 	(wire
 		(pts
-			(xy 153.67 99.06) (xy 153.67 100.33)
-		)
-		(stroke
-			(width 0)
-			(type default)
-		)
-	)
-	(wire
-		(pts
 			(xy 111.76 76.2) (xy 114.3 76.2)
 		)
@@
 	(wire
 		(pts
+			(xy 168.91 93.98) (xy 168.91 96.52)
+		)
+		(stroke
+			(width 0)
+			(type default)
+		)
+	)
+	(wire
+		(pts
 			(xy 139.7 110.49) (xy 139.7 116.84)
 		)
@@
 	(wire
 		(pts
+			(xy 151.13 91.44) (xy 156.21 91.44)
+		)
+		(stroke
+			(width 0)
+			(type default)
+		)
+	)
+	(wire
+		(pts
 			(xy 165.1 63.5) (xy 167.64 63.5)
 		)
@@
 	(wire
 		(pts
-			(xy 151.13 95.25) (xy 151.13 100.33)
+			(xy 151.13 91.44) (xy 151.13 100.33)
 		)
 		(stroke
@@
 	(wire
 		(pts
-			(xy 151.13 95.25) (xy 157.48 95.25)
-		)
-		(stroke
-			(width 0)
-			(type default)
-		)
-	)
-	(wire
-		(pts
 			(xy 111.76 50.8) (xy 114.3 50.8)
 		)
@@
 	(wire
 		(pts
+			(xy 156.21 91.44) (xy 156.21 92.71)
+		)
+		(stroke
+			(width 0)
+			(type default)
+		)
+	)
+	(wire
+		(pts
 			(xy 109.22 110.49) (xy 111.76 110.49)
 		)
@@
 	(wire
 		(pts
+			(xy 168.91 96.52) (xy 160.02 96.52)
+		)
+		(stroke
+			(width 0)
+			(type default)
+		)
+	)
+	(wire
+		(pts
 			(xy 167.64 50.8) (xy 170.18 50.8)
 		)
@@
 		(pts
 			(xy 139.7 88.9) (xy 139.7 105.41)
+		)
+		(stroke
+			(width 0)
+			(type default)
+		)
+	)
+	(wire
+		(pts
+			(xy 156.21 100.33) (xy 153.67 100.33)
 		)
 		(stroke
@@
 			)
 		)
-		(property "Footprint" "Capacitor_THT:C_Disc_D5.0mm_W2.5mm_P5.00mm"
+		(property "Footprint" "Capacitor_SMD:C_0805_2012Metric_Pad1.18x1.45mm_HandSolder"
 			(at 152.4 62.5348 0)
 			(effects
@@
 	(symbol
 		(lib_id "Device:R_Potentiometer_Trim_US")
-		(at 157.48 99.06 180)
+		(at 156.21 96.52 0)
 		(unit 1)
 		(exclude_from_sim no)
@@
 		(dnp no)
 		(property "Reference" "RV1"
-			(at 158.75 101.854 0)
+			(at 160.782 93.98 0)
 			(effects
 				(font
@@
 		)
 		(property "Value" "10k"
-			(at 157.988 94.234 0)
+			(at 161.036 99.06 0)
 			(effects
 				(font
@@
 			)
 		)
-		(property "Footprint" "Potentiometer_THT:Potentiometer_Runtron_RM-065_Vertical"
-			(at 157.48 99.06 0)
+		(property "Footprint" "Potentiometer_THT:Potentiometer_Bourns_3296W_Vertical"
+			(at 156.21 96.52 0)
 			(effects
 				(font
@@
 		)
 		(property "Datasheet" "~"
-			(at 157.48 99.06 0)
+			(at 156.21 96.52 0)
 			(effects
 				(font
@@
 		)
 		(property "Description" "Trim-potentiometer, US symbol"
-			(at 157.48 99.06 0)
+			(at 156.21 96.52 0)
 			(effects
 				(font
@@
 	)
 	(symbol
+		(lib_id "power:-15V")
+		(at 168.91 93.98 0)
+		(unit 1)
+		(exclude_from_sim no)
+		(in_bom yes)
+		(on_board yes)
+		(dnp no)
+		(property "Reference" "#PWR046"
+			(at 168.91 97.79 0)
+			(effects
+				(font
+					(size 1.27 1.27)
+				)
+				(hide yes)
+			)
+		)
+		(property "Value" "-15V"
+			(at 163.068 91.948 0)
+			(effects
+				(font
+					(size 1.27 1.27)
+				)
+				(justify left)
+			)
+		)
+		(property "Footprint" ""
+			(at 168.91 93.98 0)
+			(effects
+				(font
+					(size 1.27 1.27)
+				)
+				(hide yes)
+			)
+		)
+		(property "Datasheet" ""
+			(at 168.91 93.98 0)
+			(effects
+				(font
+					(size 1.27 1.27)
+				)
+				(hide yes)
+			)
+		)
+		(property "Description" "Power symbol creates a global label with name \"-15V\""
+			(at 168.91 93.98 0)
+			(effects
+				(font
+					(size 1.27 1.27)
+				)
+				(hide yes)
+			)
+		)
+		(pin "1"
+		)
+		(instances
+			(project "Op-Amp Training Kit"
+				(path "/5c4a903a-e3d4-449c-8c2a-618cbf16a08f/0c3d5375-59ad-4a96-9904-d4a342964cf9"
+					(reference "#PWR046")
+					(unit 1)
+				)
+			)
+		)
+	)
+	(symbol
 		(lib_id "Device:R_US")
 		(at 130.81 76.2 90)
@@
 			)
 		)
-		(property "Footprint" "Capacitor_THT:C_Disc_D5.0mm_W2.5mm_P5.00mm"
+		(property "Footprint" "Capacitor_SMD:C_0805_2012Metric_Pad1.18x1.45mm_HandSolder"
 			(at 152.4 75.2348 0)
 			(effects
@@
 			)
 		)
-		(property "Footprint" "Capacitor_THT:C_Disc_D5.0mm_W2.5mm_P5.00mm"
+		(property "Footprint" "Capacitor_SMD:C_0805_2012Metric_Pad1.18x1.45mm_HandSolder"
 			(at 152.4 87.9348 0)
 			(effects
