File: Peripheral.kicad_sch (KiCad schematic)
At the start: 0 parts

Commit message: added inverting ckt
Parts:
- added D1: LED, LED_THT:LED_D5.0mm, symbol Device:LED
- added D2: LED, LED_THT:LED_D5.0mm_Clear, symbol Device:LED
- added D3, D4: 1N4007, Diode_THT:D_DO-41_SOD81_P10.16mm_Horizontal, symbol Diode:1N4007
- added J51, J52, J53, J54, J55, J56, J57, J58: Conn_01x02_Pin, Connector_PinHeader_2.54mm:PinHeader_1x02_P2.54mm_Vertical, symbol Connector:Conn_01x02_Pin
- added R26, R27: 1k, Resistor_THT:R_Axial_DIN0207_L6.3mm_D2.5mm_P10.16mm_Horizontal, symbol Device:R_US
- added RV2: 1k, symbol Device:R_Potentiometer_US
- added RV3: 10K, symbol Device:R_Potentiometer_Trim_US
Connections:
- new net: D4.1 (K), J55.1 (Pin_1), J55.2 (Pin_2)
- new net: D1.2 (A), R26.2
- new net: J51.1 (Pin_1), J51.2 (Pin_2), R26.1
- new net: J57.1 (Pin_1), J57.2 (Pin_2), RV3.2
- new net: D3.1 (K), J56.1 (Pin_1), J56.2 (Pin_2)
- new net: D3.2 (A), J53.1 (Pin_1), J53.2 (Pin_2)
- new net: D2.2 (A), R27.2
- new net: J52.1 (Pin_1), J52.2 (Pin_2), R27.1
- new net: J58.1 (Pin_1), J58.2 (Pin_2), RV2.2
- new net: D4.2 (A), J54.1 (Pin_1), J54.2 (Pin_2)
- new net +15V: RV2.1, RV3.1
- new net GND: D1.1 (K), D2.1 (K), RV2.3, RV3.3
Other:
- note added: "Diode"
- note added: "LED"
- note added: "POT"

Commit message: Floor Planning 50%
Parts:
- RV2, RV3: footprint (none) -> Potentiometer_THT:Potentiometer_Runtron_RM-065_Vertical
Connections:
- net +15V: no longer RV2.1
- new net -15V: RV2.1
Changed lines of the file:
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@@
 			)
 		)
-		(property "Footprint" ""
+		(property "Footprint" "Potentiometer_THT:Potentiometer_Runtron_RM-065_Vertical"
 			(at 118.11 128.27 0)
 			(effects
@@
 	)
 	(symbol
+		(lib_id "power:-15V")
+		(at 152.4 125.73 0)
+		(unit 1)
+		(exclude_from_sim no)
+		(in_bom yes)
+		(on_board yes)
+		(dnp no)
+		(fields_autoplaced yes)
+		(property "Reference" "#PWR013"
+			(at 152.4 129.54 0)
+			(effects
+				(font
+					(size 1.27 1.27)
+				)
+				(hide yes)
+			)
+		)
+		(property "Value" "-15V"
+			(at 152.4 120.65 0)
+			(effects
+				(font
+					(size 1.27 1.27)
+				)
+			)
+		)
+		(property "Footprint" ""
+			(at 152.4 125.73 0)
+			(effects
+				(font
+					(size 1.27 1.27)
+				)
+				(hide yes)
+			)
+		)
+		(property "Datasheet" ""
+			(at 152.4 125.73 0)
+			(effects
+				(font
+					(size 1.27 1.27)
+				)
+				(hide yes)
+			)
+		)
+		(property "Description" "Power symbol creates a global label with name \"-15V\""
+			(at 152.4 125.73 0)
+			(effects
+				(font
+					(size 1.27 1.27)
+				)
+				(hide yes)
+			)
+		)
+		(pin "1"
+		)
+		(instances
+			(project "Op-Amp Training Kit"
+				(path "/5c4a903a-e3d4-449c-8c2a-618cbf16a08f/747d7fa1-7868-4878-b4f1-e6bff8902b26"
+					(reference "#PWR013")
+					(unit 1)
+				)
+			)
+		)
+	)
+	(symbol
 		(lib_id "Device:R_US")
 		(at 78.74 63.5 90)
@@
 	)
 	(symbol
-		(lib_id "power:+15V")
-		(at 152.4 125.73 0)
-		(unit 1)
-		(exclude_from_sim no)
-		(in_bom yes)
-		(on_board yes)
-		(dnp no)
-		(fields_autoplaced yes)
-		(property "Reference" "#PWR013"
-			(at 152.4 129.54 0)
-			(effects
-				(font
-					(size 1.27 1.27)
-				)
-				(hide yes)
-			)
-		)
-		(property "Value" "+15V"
-			(at 152.4 120.65 0)
-			(effects
-				(font
-					(size 1.27 1.27)
-				)
-			)
-		)
-		(property "Footprint" ""
-			(at 152.4 125.73 0)
-			(effects
-				(font
-					(size 1.27 1.27)
-				)
-				(hide yes)
-			)
-		)
-		(property "Datasheet" ""
-			(at 152.4 125.73 0)
-			(effects
-				(font
-					(size 1.27 1.27)
-				)
-				(hide yes)
-			)
-		)
-		(property "Description" "Power symbol creates a global label with name \"+15V\""
-			(at 152.4 125.73 0)
-			(effects
-				(font
-					(size 1.27 1.27)
-				)
-				(hide yes)
-			)
-		)
-		(pin "1"
-		)
-		(instances
-			(project "Op-Amp Training Kit"
-				(path "/5c4a903a-e3d4-449c-8c2a-618cbf16a08f/747d7fa1-7868-4878-b4f1-e6bff8902b26"
-					(reference "#PWR013")
-					(unit 1)
-				)
-			)
-		)
-	)
-	(symbol
 		(lib_id "Connector:Conn_01x02_Pin")
 		(at 167.64 60.96 270)
@@
 			)
 		)
-		(property "Footprint" ""
+		(property "Footprint" "Potentiometer_THT:Potentiometer_Runtron_RM-065_Vertical"
 			(at 146.05 128.27 0)
 			(effects
