File: Op-Amp Training Kit.kicad_pcb (KiCad board)
At the start: 2 copper layers, 145 parts, among them J1 Conn_01x04_Pin, J10 Conn_01x04_Pin, J11 Conn_01x04_Pin, J12 Conn_01x04_Pin, J13 Conn_01x04_Pin, J14 Conn_01x04_Pin, J15 Conn_01x04_Pin, J16 Conn_01x04_Pin, J17 Conn_01x04_Pin, J18 Conn_01x04_Pin, J19 Conn_01x04_Pin, J2 Conn_01x04_Pin, J20 Conn_01x04_Pin, J21 Conn_01x04_Pin, J22 Conn_01x04_Pin, J23 Conn_01x04_Pin, J24 Conn_01x04_Pin, J25 Conn_01x04_Pin, J26 Conn_01x04_Pin, J27 Conn_01x04_Pin, J28 Conn_01x04_Pin, J29 Conn_01x04_Pin, J3 Conn_01x04_Pin, J30 Conn_01x04_Pin, J31 Conn_01x04_Pin, J32 Conn_01x04_Pin, J33 Conn_01x04_Pin, J34 Conn_01x04_Pin, J35 Conn_01x04_Pin, J36 Conn_01x04_Pin, J37 Conn_01x04_Pin, J38 Conn_01x04_Pin, J39 Conn_02x04_Counter_Clockwise, J4 Conn_01x04_Pin, J40 Conn_01x04_Pin, J41 Conn_01x04_Pin, J42 Conn_01x04_Pin, J43 Conn_01x04_Pin, J44 Conn_01x04_Pin, J45 Conn_01x04_Pin, J46 Conn_01x04_Pin, J47 Conn_01x04_Pin, J48 Conn_01x04_Pin, J49 Conn_01x04_Pin, J5 Conn_01x04_Pin, J50 Conn_01x04_Pin, J51 Conn_01x02_Pin, J52 Conn_01x02_Pin, J53 Conn_01x02_Pin, J54 Conn_01x02_Pin, J55 Conn_01x02_Pin, J56 Conn_01x02_Pin, J57 Conn_01x02_Pin, J58 Conn_01x02_Pin, J59 Conn_01x04_Pin, J6 Conn_01x04_Pin, J60 Conn_01x04_Pin, J61 Conn_01x04_Pin, J62 Conn_01x04_Pin, J63 Screw_Terminal_01x03, J66 Conn_02x04_Counter_Clockwise, J67 Conn_02x04_Counter_Clockwise, J7 Conn_01x04_Pin, J8 Conn_01x04_Pin, J9 Conn_01x04_Pin, SW1 Slide Switch, SW2 Slide Switch, SW3 Slide Switch, SW4 Slide Switch, SW5 Slide Switch, SW6 Slide Switch, SW7 Slide Switch, SW8 Slide Switch, U1 LM358, U2 LM741, U3 LM741, U4 LF351N

Commit message: Completed V1
Parts:
- moved J19 237.4 mm to (166.7, 102.9), turned to 90 degrees
- moved J18 236.4 mm to (166.7, 92.8), turned to 90 degrees
- moved J28 194.1 mm to (212.6, 104.7), turned to 90 degrees
- moved J9 191.8 mm to (212.5, 97.8), turned to 90 degrees
- moved U1 172.3 mm to (213.0, 74.2)
- moved R17 171.1 mm to (174.4, 52.1), turned to 180 degrees
- moved J38 168.9 mm to (257.0, 92.8), turned to 90 degrees
- moved C3 167.9 mm to (173.3, 62.4), turned to 180 degrees
- moved J37 159.0 mm to (257.0, 103.0), turned to 90 degrees
- moved R18 147.1 mm to (174.3, 148.7), turned to 180 degrees
- moved C5 143.2 mm to (173.3, 118.2), turned to 180 degrees
- moved C6 142.9 mm to (173.3, 128.3), turned to 180 degrees
- moved C7 141.8 mm to (173.3, 138.5), turned to 180 degrees
- moved R4 136.1 mm to (194.7, 52.1), turned to 180 degrees
- moved J8 130.0 mm to (184.5, 47.0), turned to 90 degrees
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Connections:
- U1 pad 2: Net-(J19-Pin_1) -> Net-(J18-Pin_1)
- U1 pad 3: Net-(J18-Pin_1) -> Net-(J19-Pin_1)
- U1 pad 5: Net-(J38-Pin_1) -> Net-(J37-Pin_1)
- U1 pad 6: Net-(J37-Pin_1) -> Net-(J38-Pin_1)
Routing:
- net +15V: track 0.00 -> 482.9 mm
- net -15V: track 0.00 -> 458.8 mm
- net Net-(J37-Pin_1): track 0.00 -> 149.7 mm, vias 0 -> 3
- net Net-(J19-Pin_1): track 0.00 -> 142.6 mm, vias 0 -> 3
- net Net-(J38-Pin_1): track 0.00 -> 141.0 mm, vias 0 -> 3
- net Net-(J18-Pin_1): track 0.00 -> 134.4 mm, vias 0 -> 3
- net Net-(J40-Pin_1): track 0.00 -> 130.8 mm, vias 0 -> 3
- net Net-(J42-Pin_1): track 0.00 -> 49.9 mm
- net Net-(J62-Pin_1): track 0.00 -> 46.6 mm
- net Net-(J28-Pin_1): track 0.00 -> 46.2 mm
- net Net-(J60-Pin_1): track 0.00 -> 43.2 mm
- net Net-(U3-+): track 0.00 -> 36.9 mm, vias 0 -> 1
- net Net-(J9-Pin_1): track 0.00 -> 33.9 mm
- net Net-(J61-Pin_1): track 0.00 -> 30.8 mm
- net Net-(J59-Pin_1): track 0.00 -> 29.0 mm, vias 0 -> 1
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- added copper zone on B.Cu, net GND
Other:
- board outline added: 237.7 x 121.7 mm
- board text added: "0"
- board text added: "1"
- board text added: "2"
- board text added: "3"
- board text added: "4"
- board text added: "5"
- board text added: "6"
- board text added: "7"
- board text added: "8-bit DAC"
- board text added: "Basic Op-Amp"
- board text added: "Diode"
- board text added: "Full Op-Amp"
- board text added: "Inverting Op-Amp"
- board text added: "LED"
- board text added: "LSB"
- board text added: "MSB"
- board text added: "Potentiometer"

Commit message: Updated track
Routing:
- net +15V: track 482.9 -> 481.8 mm
Changed lines of the file:
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@@
+	)
+	(segment
+		(start 94.14 57.34)
+		(end 92.4 55.6)
+		(width 1.524)
+		(layer "B.Cu")
+		(net 23)
+	)
+	(segment
+		(start 155.55 50.75)
+		(end 155.55 56.1844)
+		(width 1.27)
+		(layer "B.Cu")
+		(net 23)
+	)
+	(segment
+		(start 165.05 41.25)
+		(end 155.55 50.75)
+		(width 1.27)
+		(layer "B.Cu")
+		(net 23)
+	)
+	(segment
+		(start 46.2285 62.484)
+		(end 51.308 62.484)
+		(width 2.54)
+		(layer "B.Cu")
+		(net 23)
+	)
+	(segment
+		(start 65 96)
+		(end 67 98)
+		(width 2.032)
+		(layer "B.Cu")
+		(net 23)
+	)
+	(segment
+		(start 77.3684 40.0304)
+		(end 75.438 41.9608)
+		(width 1.524)
+		(layer "B.Cu")
+		(net 23)
+	)
+	(segment
+		(start 92.4052 55.5244)
+		(end 92.4052 42.7736)
+		(width 1.524)
+		(layer "B.Cu")
+		(net 23)
+	)
+	(segment
+		(start 57.15 69.85)
+		(end 57.404 70.104)
+		(width 1.524)
+		(layer "B.Cu")
+		(net 23)
+	)
+	(segment
+		(start 59 96)
+		(end 65 96)
+		(width 2.032)
+		(layer "B.Cu")
+		(net 23)
+	)
+	(segment
+		(start 58.928 62.484)
+		(end 51.308 62.484)
+		(width 2.54)
+		(layer "B.Cu")
+		(net 23)
+	)
+	(segment
+		(start 67 98)
+		(end 67 116.34)
+		(width 2.032)
+		(layer "B.Cu")
+		(net 23)
+	)
+	(segment
+		(start 57.15 63.246)
+		(end 56.388 62.484)
+		(width 2.032)
+		(layer "B.Cu")
+		(net 23)
+	)
+	(segment
+		(start 138.4616 114.2884)
+		(end 138.4616 124.1426)
+		(width 1.27)
+		(layer "B.Cu")
+		(net 23)
+	)
+	(segment
+		(start 54 91)
+		(end 59 96)
+		(width 2.032)
+		(layer "B.Cu")
+		(net 23)
+	)
+	(segment
+		(start 41.5665 57.822)
+		(end 46.2285 62.484)
+		(width 2.54)
+		(layer "B.Cu")
+		(net 23)
+	)
+	(segment
+		(start 92.4 55.6)
+		(end 92.4 55.5296)
+		(width 1.524)
+		(layer "B.Cu")
+		(net 23)
+	)
+	(segment
+		(start 54 77)
+		(end 54 91)
+		(width 2.032)
+		(layer "B.Cu")
+		(net 23)
+	)
+	(segment
+		(start 220.65 59.5)
+		(end 202.4 41.25)
+		(width 1.27)
+		(layer "B.Cu")
+		(net 23)
+	)
+	(segment
+		(start 75.438 44.9072)
+		(end 79.248 48.7172)
+		(width 1.524)
+		(layer "B.Cu")
+		(net 23)
+	)
+	(segment
+		(start 51.308 59.944)
+		(end 51.308 62.484)
+		(width 2.54)
+		(layer "B.Cu")
+		(net 23)
+	)
+	(segment
+		(start 220.65 74.17)
+		(end 220.65 59.5)
+		(width 1.27)
+		(layer "B.Cu")
+		(net 23)
+	)
+	(segment
+		(start 65.17 118.17)
+		(end 65.17 123.73)
+		(width 2.032)
+		(layer "B.Cu")
+		(net 23)
+	)
+	(segment
+		(start 57.15 75.184)
+		(end 57.15 69.85)
+		(width 2.032)
+		(layer "B.Cu")
+		(net 23)
+	)
+	(segment
+		(start 155.446 70.104)
+		(end 155.55 70)
+		(width 1.524)
+		(layer "B.Cu")
+		(net 23)
+	)
+	(segment
+		(start 96.012 57.34)
+		(end 94.14 57.34)
+		(width 1.524)
+		(layer "B.Cu")
+		(net 23)
+	)
+	(segment
+		(start 92.4052 42.7736)
+		(end 89.662 40.0304)
+		(width 1.524)
+		(layer "B.Cu")
+		(net 23)
+	)
+	(segment
+		(start 58.928 59.944)
+		(end 58.928 62.484)
+		(width 2.54)
+		(layer "B.Cu")
+		(net 23)
+	)
+	(segment
+		(start 57.15 75.184)
+		(end 55.816 75.184)
+		(width 2.032)
+		(layer "B.Cu")
+		(net 23)
 	)
 	(segment
@@
 	)
 	(segment
-		(start 155.55 50.75)
-		(end 155.55 56.1844)
-		(width 1.27)
-		(layer "B.Cu")
-		(net 23)
-	)
-	(segment
-		(start 165.05 41.25)
-		(end 155.55 50.75)
-		(width 1.27)
-		(layer "B.Cu")
-		(net 23)
-	)
-	(segment
-		(start 46.2285 62.484)
-		(end 51.308 62.484)
-		(width 2.54)
-		(layer "B.Cu")
-		(net 23)
-	)
-	(segment
-		(start 65 96)
-		(end 67 98)
-		(width 2.032)
-		(layer "B.Cu")
-		(net 23)
-	)
-	(segment
-		(start 57.15 69.85)
-		(end 57.404 70.104)
-		(width 1.524)
-		(layer "B.Cu")
-		(net 23)
-	)
-	(segment
-		(start 92.4052 55.5244)
-		(end 92.4052 42.7736)
-		(width 1.524)
-		(layer "B.Cu")
-		(net 23)
-	)
-	(segment
-		(start 59 96)
-		(end 65 96)
-		(width 2.032)
-		(layer "B.Cu")
-		(net 23)
-	)
-	(segment
-		(start 58.928 62.484)
-		(end 51.308 62.484)
-		(width 2.54)
-		(layer "B.Cu")
-		(net 23)
-	)
-	(segment
-		(start 93.1032 57.34)
-		(end 91.8464 56.0832)
-		(width 1.524)
-		(layer "B.Cu")
-		(net 23)
-	)
-	(segment
-		(start 67 98)
-		(end 67 116.34)
-		(width 2.032)
-		(layer "B.Cu")
-		(net 23)
-	)
-	(segment
-		(start 57.15 63.246)
-		(end 56.388 62.484)
-		(width 2.032)
-		(layer "B.Cu")
-		(net 23)
-	)
-	(segment
-		(start 138.4616 114.2884)
-		(end 138.4616 124.1426)
-		(width 1.27)
-		(layer "B.Cu")
-		(net 23)
-	)
-	(segment
-		(start 54 91)
-		(end 59 96)
-		(width 2.032)
-		(layer "B.Cu")
-		(net 23)
-	)
-	(segment
-		(start 41.5665 57.822)
-		(end 46.2285 62.484)
-		(width 2.54)
-		(layer "B.Cu")
-		(net 23)
-	)
-	(segment
-		(start 54 77)
-		(end 54 91)
-		(width 2.032)
-		(layer "B.Cu")
-		(net 23)
-	)
-	(segment
-		(start 220.65 59.5)
-		(end 202.4 41.25)
-		(width 1.27)
-		(layer "B.Cu")
-		(net 23)
-	)
-	(segment
-		(start 77.3684 40.0304)
-		(end 75.438 41.9608)
-		(width 1.524)
-		(layer "B.Cu")
-		(net 23)
-	)
-	(segment
-		(start 51.308 59.944)
-		(end 51.308 62.484)
-		(width 2.54)
-		(layer "B.Cu")
-		(net 23)
-	)
-	(segment
-		(start 220.65 74.17)
-		(end 220.65 59.5)
-		(width 1.27)
-		(layer "B.Cu")
-		(net 23)
-	)
-	(segment
-		(start 65.17 118.17)
-		(end 65.17 123.73)
-		(width 2.032)
-		(layer "B.Cu")
-		(net 23)
-	)
-	(segment
-		(start 57.15 75.184)
-		(end 57.15 69.85)
-		(width 2.032)
-		(layer "B.Cu")
-		(net 23)
-	)
-	(segment
-		(start 155.446 70.104)
-		(end 155.55 70)
-		(width 1.524)
-		(layer "B.Cu")
-		(net 23)
-	)
-	(segment
-		(start 58.928 59.944)
-		(end 58.928 62.484)
-		(width 2.54)
-		(layer "B.Cu")
-		(net 23)
-	)
-	(segment
-		(start 57.15 75.184)
-		(end 55.816 75.184)
-		(width 2.032)
-		(layer "B.Cu")
-		(net 23)
-	)
-	(segment
 		(start 154.3812 57.3532)
 		(end 154.368 57.34)
@@
 	)
 	(segment
-		(start 96.012 57.34)
-		(end 93.1032 57.34)
-		(width 1.524)
-		(layer "B.Cu")
-		(net 23)
-	)
-	(segment
 		(start 202.4 41.25)
 		(end 165.05 41.25)
@@
 	)
 	(segment
+		(start 75.438 41.9608)
+		(end 75.438 44.9072)
+		(width 1.524)
+		(layer "B.Cu")
+		(net 23)
+	)
+	(segment
+		(start 92.4 55.5296)
+		(end 92.4052 55.5244)
+		(width 1.524)
+		(layer "B.Cu")
+		(net 23)
+	)
+	(segment
 		(start 96.012 57.34)
 		(end 149.352 57.34)
@@
 	)
 	(segment
-		(start 75.438 44.9072)
-		(end 79.248 48.7172)
-		(width 1.524)
-		(layer "B.Cu")
-		(net 23)
-	)
-	(segment
-		(start 75.438 41.9608)
-		(end 75.438 44.9072)
-		(width 1.524)
-		(layer "B.Cu")
-		(net 23)
-	)
-	(segment
 		(start 154.368 57.34)
 		(end 149.352 57.34)
@@
 	)
 	(segment
-		(start 92.4052 42.7736)
-		(end 89.662 40.0304)
-		(width 1.524)
-		(layer "B.Cu")
-		(net 23)
-	)
-	(segment
 		(start 155.55 70)
 		(end 155.55 97.2)
@@
 		(layer "B.Cu")
 		(net 23)
-	)
-	(segment
-		(start 91.8464 56.0832)
-		(end 92.4052 55.5244)
-		(width 1.524)
-		(layer "B.Cu")
-		(net 23)

Commit message: Filanl Pakka
Parts:
- C1, C10, C11, C12, C13, C14, C15, C2, C3, C4, C5, C6, C7, C8, C9, R28, R29, R30, R31, R32, R33, R34, R35, R36, R37, R38, R39, R40, R41, R42, R43, R44: moved to B.Cu
- moved J9 4.55 mm to (212.6, 93.3)
- moved C5 0.57 mm to (172.8, 118.2)
- moved C3 0.18 mm to (173.3, 62.2)
- moved R43 0.10 mm to (142.8, 42.2)
- moved R31 0.10 mm to (104.7, 42.2)
- moved C4 0.09 mm to (105.7, 124.9)
- moved C2 0.09 mm to (173.4, 72.5)
- moved R29 0.08 mm to (97.0, 42.2)
- moved R40 0.07 mm to (119.9, 42.2)
- moved R42 0.07 mm to (135.1, 42.2)
- moved R41 0.07 mm to (127.5, 42.2)
- moved C7 0.06 mm to (173.3, 138.5)
- moved C10 0.05 mm to (258.0, 62.3)
- moved C12 0.05 mm to (258.0, 82.7)
Routing:
- net +15V: track 481.8 -> 490.1 mm
- net GND: track 27.3 -> 21.4 mm, vias 2 -> 4
- net Net-(J9-Pin_1): track 33.9 -> 29.4 mm
- net -15V: track 458.8 -> 461.1 mm
- net Net-(J22-Pin_1): track 18.2 -> 16.4 mm, vias 1 -> 0
- net Net-(U3-+): track 36.9 -> 38.7 mm, vias 1 -> 2
- net Net-(J23-Pin_1): track 18.5 -> 17.3 mm, vias 1 -> 0
- net Net-(J10-Pin_1): track 18.2 -> 17.1 mm, vias 1 -> 0
- net Net-(J24-Pin_1): track 18.2 -> 17.2 mm, vias 1 -> 0
- net Net-(J19-Pin_1): track 142.6 -> 143.6 mm, vias 3 -> 0
- net Net-(J43-Pin_1): track 18.2 -> 17.3 mm, vias 1 -> 0
- net Net-(J4-Pin_1): track 18.3 -> 17.4 mm, vias 1 -> 0
- net Net-(J12-Pin_1): track 18.3 -> 17.4 mm, vias 1 -> 0
- net Net-(J11-Pin_1): track 18.2 -> 17.4 mm, vias 1 -> 0
- net Net-(J25-Pin_1): track 18.2 -> 17.4 mm, vias 1 -> 0
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Other:
- outline, holes or cut-outs redrawn
