File: Op-Amp Training Kit.kicad_pcb (KiCad board)
At the start: 2 copper layers, 237.7 x 121.7 mm, 145 parts, among them J1 Conn_01x04_Pin, J10 Conn_01x04_Pin, J11 Conn_01x04_Pin, J12 Conn_01x04_Pin, J13 Conn_01x04_Pin, J14 Conn_01x04_Pin, J15 Conn_01x04_Pin, J16 Conn_01x04_Pin, J17 Conn_01x04_Pin, J18 Conn_01x04_Pin, J19 Conn_01x04_Pin, J2 Conn_01x04_Pin, J20 Conn_01x04_Pin, J21 Conn_01x04_Pin, J22 Conn_01x04_Pin, J23 Conn_01x04_Pin, J24 Conn_01x04_Pin, J25 Conn_01x04_Pin, J26 Conn_01x04_Pin, J27 Conn_01x04_Pin, J28 Conn_01x04_Pin, J29 Conn_01x04_Pin, J3 Conn_01x04_Pin, J30 Conn_01x04_Pin, J31 Conn_01x04_Pin, J32 Conn_01x04_Pin, J33 Conn_01x04_Pin, J34 Conn_01x04_Pin, J35 Conn_01x04_Pin, J36 Conn_01x04_Pin, J37 Conn_01x04_Pin, J38 Conn_01x04_Pin, J39 Conn_02x04_Counter_Clockwise, J4 Conn_01x04_Pin, J40 Conn_01x04_Pin, J41 Conn_01x04_Pin, J42 Conn_01x04_Pin, J43 Conn_01x04_Pin, J44 Conn_01x04_Pin, J45 Conn_01x04_Pin, J46 Conn_01x04_Pin, J47 Conn_01x04_Pin, J48 Conn_01x04_Pin, J49 Conn_01x04_Pin, J5 Conn_01x04_Pin, J50 Conn_01x04_Pin, J51 Conn_01x02_Pin, J52 Conn_01x02_Pin, J53 Conn_01x02_Pin, J54 Conn_01x02_Pin, J55 Conn_01x02_Pin, J56 Conn_01x02_Pin, J57 Conn_01x02_Pin, J58 Conn_01x02_Pin, J59 Conn_01x04_Pin, J6 Conn_01x04_Pin, J60 Conn_01x04_Pin, J61 Conn_01x04_Pin, J62 Conn_01x04_Pin, J63 Screw_Terminal_01x03, J66 Conn_02x04_Counter_Clockwise, J67 Conn_02x04_Counter_Clockwise, J7 Conn_01x04_Pin, J8 Conn_01x04_Pin, J9 Conn_01x04_Pin, SW1 Slide Switch, SW2 Slide Switch, SW3 Slide Switch, SW4 Slide Switch, SW5 Slide Switch, SW6 Slide Switch, SW7 Slide Switch, SW8 Slide Switch, U1 LM358, U2 LM741, U3 LM741, U4 LF351N

Commit message: Changes in Silkscreen
Other:
- board text added: "BJT type Slew Rate 0.5v/us GWB 1MHz CMMR 90dB"
- board text added: "Dual op amp BJT type Slew Rate 0.3V/us GWB 1MHz"
- board text added: "JFET type Slew Rate 13V/us GWB 13MHz"
- board text added: "This Op-Amp can be programmed in any configuration with pre-installed resistors and capacitors"
- board text added: "This Op-Amp stays in inverting state i.e non-inverting terminal is connected to GND"
